File: kicad/attiny-modulator.kicad_sch (KiCad schematic)
At the start: 5 parts, among them J1 Eurorack Power Large, U1 ATtiny85-20M, U2 L7805

Commit message: Updating schematic, layout and front panel
Parts:
- removed J1: Eurorack Power Large, Eurorack_Power:Eurorack_PowerHeader_2x08_P2.54mm_Shrouded, symbol Eurorack_Power:Eurorack Power Large
- removed U1: ATtiny85-20M, Package_DFN_QFN:QFN-20-1EP_4x4mm_P0.5mm_EP2.6x2.6mm, symbol MCU_Microchip_ATtiny:ATtiny85-20M
- removed U2: L7805, symbol Regulator_Linear:L7805
- added C1, C10, C2, C6, C7, C8: 100nF, Rumblesan_Standard_Parts:C_Rect_L7.0mm_W2.5mm_P5.00mm, symbol Rumblesan Standard Parts:C
- added C12, C4: 1nF, Rumblesan_Standard_Parts:C_Rect_L7.0mm_W2.5mm_P5.00mm, symbol Rumblesan Standard Parts:C
- added C3, C5: 10uF, Rumblesan_Standard_Parts:CP_Radial_D5.0mm_P2.00mm, symbol Rumblesan Standard Parts:C_Polarized
- added C9: 1n8F, Rumblesan_Standard_Parts:C_Rect_L7.0mm_W3.5mm_P5.00mm, symbol Rumblesan Standard Parts:C
- added D3, D4, D5: LED, LED_THT:LED_D1.8mm_W3.3mm_H2.4mm, symbol Device:LED
- added D6: 1N4148, Rumblesan_Standard_Parts:D_DO-35_SOD27_P7.62mm_Horizontal, symbol Device:D
- added H1, H2, H3, H4: MountingHole_Pad, MountingHole:MountingHole_3.2mm_M3_DIN965_Pad, symbol Mechanical:MountingHole_Pad
- added J1: Eurorack Power Small, Eurorack_Power:Eurorack_PowerHeader_2x05_P2.54mm_Shrouded, symbol Eurorack_Power:Eurorack Power Small
- added J10, J7: Conn_01x04_Socket, Connector_PinSocket_2.54mm:PinSocket_1x04_P2.54mm_Vertical, symbol Connector:Conn_01x04_Socket
- added J11, J2, J3, J4, J5: Eurorack Mono Jack, Rumblesan_Standard_Parts:Jack_3.5mm_QingPu_WQP-PJ398SM_Vertical, symbol Audio_Connectors:Eurorack_Mono_Jack
- added J12: Conn_01x05_Pin, Connector_PinHeader_2.54mm:PinHeader_1x05_P2.54mm_Vertical, symbol Connector:Conn_01x05_Pin
- added J13: Conn_01x05_Socket, Connector_PinSocket_2.54mm:PinSocket_1x05_P2.54mm_Vertical, symbol Connector:Conn_01x05_Socket
- added J6: AVR-ISP-6, Connector_PinHeader_2.54mm:PinHeader_2x03_P2.54mm_Vertical, symbol Connector:AVR-ISP-6
- added J8, J9: Conn_01x04_Pin, Connector_PinHeader_2.54mm:PinHeader_1x04_P2.54mm_Vertical, symbol Connector:Conn_01x04_Pin
- added JP2, JP3: Jumper_2_Open, Connector_PinHeader_2.54mm:PinHeader_1x02_P2.54mm_Vertical, symbol Jumper:Jumper_2_Open
- added Q1, Q2, Q3: BC547, Package_TO_SOT_THT:TO-92_Inline_Wide, symbol Transistor_BJT:BC547
- added R1, R2, R24, R25, R3, R4: 200k, Rumblesan_Standard_Parts:R_Axial_DIN0207_L6.3mm_D2.5mm_P10.16mm_Horizontal, symbol Rumblesan Standard Parts:R
- added R10, R11, R18, R20, R22, R26, R5, R7, R8, R9: 100k, Rumblesan_Standard_Parts:R_Axial_DIN0207_L6.3mm_D2.5mm_P10.16mm_Horizontal, symbol Rumblesan Standard Parts:R
- added R13, R19: 10k, Rumblesan_Standard_Parts:R_Axial_DIN0207_L6.3mm_D2.5mm_P10.16mm_Horizontal, symbol Rumblesan Standard Parts:R
- added R17, R6: 1k, Rumblesan_Standard_Parts:R_Axial_DIN0207_L6.3mm_D2.5mm_P10.16mm_Horizontal, symbol Rumblesan Standard Parts:R
- added R21: 47k, Rumblesan_Standard_Parts:R_Axial_DIN0207_L6.3mm_D2.5mm_P10.16mm_Horizontal, symbol Rumblesan Standard Parts:R
- added R23: R_led, Rumblesan_Standard_Parts:R_Axial_DIN0207_L6.3mm_D2.5mm_P10.16mm_Horizontal, symbol Rumblesan Standard Parts:R
- added RV1, RV2, RV3: 10k, Rumblesan_Standard_Parts:Potentiometer_Alpha_RD901F-40-00D_Single_Vertical, symbol Rumblesan Standard Parts:R_Potentiometer
- added U1: ATtiny85-20P, Package_DIP:DIP-8_W7.62mm, symbol MCU_Microchip_ATtiny:ATtiny85-20P
- added U2: MCP602, Package_DIP:DIP-8_W7.62mm_Socket, symbol Amplifier_Operational:MCP602
- added U4: L78L05_TO92, Package_TO_SOT_THT:TO-92_Inline_Wide, symbol Regulator_Linear:L78L05_TO92
- added U5: L79L05_TO92, Package_TO_SOT_THT:TO-92_Inline_Wide, symbol Regulator_Linear:L79L05_TO92
- added U6: TL072, Package_DIP:DIP-8_W7.62mm, symbol Amplifier_Operational:TL072
- D1, D2: value D_Schottky -> 1N5158; footprint (none) -> Rumblesan_Standard_Parts:D_DO-41_SOD81_P10.16mm_Horizontal
Connections:
- net GND: now also C1.2, C10.2, C2.1, C3.2, C5.1, C6.2, C7.2, C8.1, C9.1, D5.1 (K), D6.2 (A), H1.1, H2.1, H3.1, H4.1, J1.3 (GND), J1.4 (GND), J1.5 (GND), J1.6 (GND), J1.7 (GND), J1.8 (GND), J10.2 (Pin_2), J10.3 (Pin_3), J11.1 (Sleeve), J2.1 (Sleeve), J2.3 (Tip_normalize), J3.1 (Sleeve), J4.1 (Sleeve), J5.1 (Sleeve), J5.3 (Tip_normalize), J6.6 (GND), J9.2 (Pin_2), J9.3 (Pin_3), R19.2, R8.2, RV3.1, U1.4 (GND), U2.3 (+), U2.4 (V-), U2.5 (+), U4.2 (GND), U5.1 (GND), U6.6 (-)
- net at D1.2 (A): now also J1.10 (+12V), J1.9 (+12V)
- net at D2.1 (K): now also J1.1 (-12V), J1.2 (-12V)
- net +12V renamed VCC
- net VCC: now also C3.1, C7.1, U4.3 (VI), U6.8 (V+)
- net -12V renamed VEE
- net VEE: now also C5.2, C8.2, U5.2 (VI), U6.4 (V-)
- new net: J11.2 (Tip), J4.2 (Tip), R17.1
- new net: JP2.2 (B), R13.2
- new net: C4.1, R1.1, R2.1, R4.1, R5.2, U2.2 (-)
- new net: Q1.1 (C), Q2.2 (B), R20.2
- new net: Q1.3 (E), Q2.3 (E), R19.1
- new net: Q3.1 (C), R23.1
- new net: JP3.2 (B), R10.1, R9.2, U6.2 (-)
- new net: C9.2, R11.1, U6.3 (+)
- new net: D6.1 (K), Q1.2 (B), R18.1
- new net: C12.1, R24.1, R25.1, R26.2, R3.1, U2.6 (-)
- new net: J3.2 (Tip), R18.2
- new net: D5.2 (A), Q3.3 (E)
- new net: Q3.2 (B), R22.1
- new net +5V: C1.1, C10.1, C6.1, J10.1 (Pin_1), J6.2 (VCC), J9.1 (Pin_1), R10.2, R20.1, R21.1, R23.2, R7.2, RV1.3, RV2.3, RV3.3, U1.8 (VCC), U2.8 (V+), U4.1 (VO)
- new net -5V: C2.2, J10.4 (Pin_4), J9.4 (Pin_4), R25.2, R4.2, RV1.1, RV2.1, U5.3 (VO)
- new net CV1_CTRL: J13.3 (Pin_3), J5.2 (Tip)
- new net CV1_MAIN: J12.3 (Pin_3), R1.2
- new net CV2_CTRL: J13.4 (Pin_4), J2.2 (Tip)
- new net CV2_MAIN: J12.4 (Pin_4), R24.2
- new net LED_NEG_CTRL: D3.1 (K), D4.2 (A), J13.1 (Pin_1)
- new net LED_NEG_MAIN: J12.1 (Pin_1), R6.2, U6.5 (+)
- new net LED_POS_CTRL: D3.2 (A), D4.1 (K), J13.2 (Pin_2)
- new net LED_POS_MAIN: J12.2 (Pin_2), U6.7
- new net MCU_ADC_1: C4.2, J6.3 (SCK), R5.1, U1.7 (PB2), U2.1
- new net MCU_ADC_2: C12.2, R26.1, U1.3 (XTAL2/PB4), U2.7
- new net MCU_ADC_3: J8.3 (Pin_3), U1.2 (XTAL1/PB3)
- new net MCU_PWM: J6.1 (MISO), JP2.1 (A), R11.2, R8.1, U1.6 (PB1)
- new net MCU_RESET: J6.5 (~{RST}), R7.1, U1.1 (~{RESET}/PB5)
- new net MCU_TRIG: J6.4 (MOSI), J8.4 (Pin_4), U1.5 (AREF/PB0)
- new net OUT_CTRL: J13.5 (Pin_5), R17.2
- new net OUT_MAIN: J12.5 (Pin_5), JP3.1 (A), R13.1, R6.1, R9.1, U6.1
- new net POT1_CTRL: J7.1 (Pin_1), RV1.2
- new net POT1_MAIN: J8.1 (Pin_1), R2.2
- new net POT2_CTRL: J7.2 (Pin_2), RV2.2
- new net POT2_MAIN: J8.2 (Pin_2), R3.2
- new net POT3_CTRL: J7.3 (Pin_3), RV3.2
- new net TRIG_CTRL: J7.4 (Pin_4), Q2.1 (C), R21.2, R22.2
- no-connect marks 1 -> 3

Commit message: Fixing bugs with circuit
Parts:
- removed JP2, JP3: Jumper_2_Open, Connector_PinHeader_2.54mm:PinHeader_1x02_P2.54mm_Vertical, symbol Jumper:Jumper_2_Open
- removed R13: 10k, Rumblesan_Standard_Parts:R_Axial_DIN0207_L6.3mm_D2.5mm_P10.16mm_Horizontal, symbol Rumblesan Standard Parts:R
- removed R8: 100k, Rumblesan_Standard_Parts:R_Axial_DIN0207_L6.3mm_D2.5mm_P10.16mm_Horizontal, symbol Rumblesan Standard Parts:R
- added C12: 2.2nF, Rumblesan_Standard_Parts:C_Rect_L7.0mm_W3.5mm_P5.00mm, symbol Rumblesan Standard Parts:C
- added R11: 22k, Rumblesan_Standard_Parts:R_Axial_DIN0207_L6.3mm_D2.5mm_P10.16mm_Horizontal, symbol Rumblesan Standard Parts:R
- C11: renamed from C9; value 1n8F -> 1nF
- R12: renamed from R11; value 100k -> 22k
- renumbered C12 to C9
Connections:
- net GND: now also U6.5 (+); no longer U6.6 (-)
- net LED_NEG_MAIN: now also U6.6 (-); no longer U6.5 (+)
- net MCU_PWM: now also R11.1; no longer R12.2
- net OUT_MAIN: now also C12.1
- net at R12.1, U6.3 (+): no longer C11.2
- new net: C11.2, C12.2, R11.2, R12.2
Other:
- note added: "For unipolar, 0V-5V outputs, don't place R10 and place a wire jumper for R10 For bipolar, -5V-5V outputs, place both R9 and R10"
- note added: "Gain = (R10 + R9)/R10 FSF × fc = 1/(2π sqrt(R11*R12*C11*C12) Q = sqrt(R11*R12*C11*C12)/(R11*C11 + R12*C11 + R11*C12(1 − Gain)) Using ratios to make things easier to design R11 = mR , R12 = R , C11 = C , C12 = nC Q = sqrt(mn)/(m + 1 + mn(1-gain)) FSF * fc = 1/(2piRC * sqrt(mn)) For a Second-Order Low-Pass Butterworth Filter FSF = 1 Q = 0.707 if Gain = 1, then m = 1 and n = 2 gives Q of 0.707 if Ga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"
- note added: "Values shown are for Unipolar 0V-5V output For a bipolar, -5V-5V output R12 should be 47k and C12 should be 1nF"
- moved on the sheet: C11, C6, C7, C8, R10, R12, R6, R9, U2C, U6A, U6B, U6C

Commit message: Tweaks for rev02
Other:
- note added: "D4 lights on positive output D3 lights on negative output"
- note added: "For unipolar, 0V-5V outputs, don't place R10 and place a wire jumper for R9 For bipolar, -5V-5V outputs, place both R9 and R10"
- note removed: "For unipolar, 0V-5V outputs, don't place R10 and place a wire jumper for R10 For bipolar, -5V-5V outputs, place both R9 and R10"
Changed lines of the file:
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@@
   (paper "A3")
   (title_block
+    (date "2023-07-19")
+    (rev "rev02")
     (comment 1 "Based on the JNTUB designed by Ben Reeves")
     (comment 2 "creativecommons.org/licenses/by/4.0/")
@@
     (stroke (width 0) (type default))
   )
-  (text "For unipolar, 0V-5V outputs, don't place R10 and place a wire jumper for R10\nFor bipolar, -5V-5V outputs, place both R9 and R10"
+  (text "D4 lights on positive output\nD3 lights on negative output"
+    (at 99.06 158.75 0)
+    (effects (font (size 1.27 1.27)) (justify left bottom))
+  )
+  (text "For unipolar, 0V-5V outputs, don't place R10 and place a wire jumper for R9\nFor bipolar, -5V-5V outputs, place both R9 and R10"
     (at 270.51 218.44 0)
     (effects (font (size 1.27 1.27)) (justify left bottom))

Commit message: Refreshing board layout
Parts:
- C1, C10, C2, C4, C6, C7, C8, C9: symbol Rumblesan Standard Parts:C -> Standard_Parts:C
- C11, C12: footprint Rumblesan_Standard_Parts:C_Rect_L7.0mm_W3.5mm_P5.00mm -> Rumblesan_Standard_Parts:C_Rect_L7.0mm_W2.5mm_P5.00mm; symbol Rumblesan Standard Parts:C -> Standard_Parts:C
- C3, C5: symbol Rumblesan Standard Parts:C_Polarized -> Standard_Parts:C_Polarized
- H1, H2, H3, H4: now left out of the parts list
- J1: footprint Eurorack_Power:Eurorack_PowerHeader_2x05_P2.54mm_Shrouded -> Rumblesan_Eurorack_Power:Eurorack_PowerHeader_2x05_P2.54mm_Shrouded; symbol Eurorack_Power:Eurorack Power Small -> Rumblesan_Eurorack_Power:Eurorack Power Small
- J11, J2, J3, J4, J5: footprint Rumblesan_Standard_Parts:Jack_3.5mm_QingPu_WQP-PJ398SM_Vertical -> Rumblesan_Audio_Connectors:Jack_3.5mm_QingPu_WQP-PJ398SM_Vertical; symbol Audio_Connectors:Eurorack_Mono_Jack -> Connector_Audio:AudioJack2_SwitchT
- R1, R10, R11, R12, R17, R18, R19, R2, R20, R21, R22, R23, R24, R25, R26, R3, R4, R5, R6, R7, R9: symbol Rumblesan Standard Parts:R -> Standard_Parts:R
- RV1, RV2, RV3: footprint Rumblesan_Standard_Parts:Potentiometer_Alpha_RD901F-40-00D_Single_Vertical -> Rumblesan_Potentiometer_THT:Potentiometer_Alpha_RD901F-40-00D_Single_Vertical; symbol Rumblesan Standard Parts:R_Potentiometer -> Standard_Parts:R_Potentiometer
- U1, U6: footprint Package_DIP:DIP-8_W7.62mm -> Package_DIP:DIP-8_W7.62mm_Socket
Connections:
- net CV1_CTRL: now also J5.T; no longer J5.2 (Tip)
- net CV2_CTRL: now also J2.T; no longer J2.2 (Tip)
- net GND: now also J11.S, J2.S, J2.TN, J3.S, J4.S, J5.S, J5.TN; no longer J11.1 (Sleeve), J2.1 (Sleeve), J2.3 (Tip_normalize), J3.1 (Sleeve), J4.1 (Sleeve), J5.1 (Sleeve), J5.3 (Tip_normalize)
- net at R18.2: now also J3.T; no longer J3.2 (Tip)
- new net: J11.T, J4.T, R17.1
Other:
- company: (none) -> Bristol Communal Modular
- title: (none) -> ATTiny Modulator
- moved on the sheet: J11, J4
